File: current/Messwerte_nur_Strom.sch (KiCad schematic (older format))
At the start: 9 parts, among them J1 Stromsensor_01, J2 Addr, J3 Stromsensor_02, J4 Stromsensor_03, J5 Stromsensor_04, J6 I2C_Conn_12V, U1 P82B96

Commit message: pcb actualized
Signed-off-by: Samira-I2C <franz.siegele@gmx.net>
Parts:
- removed J1: Stromsensor_01, symbol Connector:Conn_01x03_Female
- removed J3: Stromsensor_02, symbol Connector:Conn_01x03_Female
- removed J4: Stromsensor_03, symbol Connector:Conn_01x03_Female
- removed J5: Stromsensor_04, symbol Connector:Conn_01x03_Female
- removed J6: I2C_Conn_12V, Connector_PinSocket_2.54mm:PinSocket_1x04_P2.54mm_Vertical, symbol Connector:Conn_01x04_Female
- removed R1, R2: 3k9, Resistor_THT:R_Axial_DIN0207_L6.3mm_D2.5mm_P10.16mm_Horizontal, symbol Device:R
- removed U1: P82B96, symbol Interface_Expansion:P82B96
- added J1: Stromsensor_01, symbol Connector:Conn_01x03_Male
- added J2: Stromsensor_02, symbol Connector:Conn_01x03_Male
- added J4: Stromsensor_03, symbol Connector:Conn_01x03_Male
- added J5: Stromsensor_04, symbol Connector:Conn_01x03_Male
- added J6: I2C/5V, symbol Connector:Conn_01x04_Male
- renumbered J2 to J3
Connections:
- net labels added: +5V
- net labels removed: +12V
- wire segments 79 -> 48
Other:
- note removed: "DCDC Wandler"
- moved on the sheet: J3
