File: volt/ADS1115.sch (KiCad schematic (older format))
At the start: 1 part, among them U2 ADS1115IDGS

Commit message: pcb actualized
Signed-off-by: Samira-I2C <franz.siegele@gmx.net>
Parts:
- renumbered U2 to U4
Changed lines of the file:
@@
 $Descr A4 11693 8268
 encoding utf-8
-Sheet 3 3
+Sheet 3 2
 Title ""
 Date ""
@@
 $EndDescr
 $Comp
-L Analog_ADC:ADS1115IDGS U2
+L Analog_ADC:ADS1115IDGS U4
 U 1 1 5E458702
 P 5550 3700
-AR Path="/5E1F6B8F/5E458702" Ref="U2"  Part="1"
+AR Path="/5E1F6B8F/5E458702" Ref="U4"  Part="1"
 AR Path="/5E339291/5E458702" Ref="U?"  Part="1"
-F 0 "U2" H 5550 4381 50  0000 C CNN
+F 0 "U4" H 5550 4381 50  0000 C CNN
 F 1 "ADS1115IDGS" H 5550 4290 50  0000 C CNN
 F 2 "Package_SO:TSSOP-10_3x3mm_P0.5mm" H 5550 3200 50  0001 C CNN

Commit message: update electronic circuit
Signed-off-by: Samira-I2C <franz.siegele@gmx.net>
Parts:
- renumbered U4 to U7
Changed lines of the file:
@@
 $Descr A4 11693 8268
 encoding utf-8
-Sheet 3 2
+Sheet 2 2
 Title ""
 Date ""
@@
 $EndDescr
 $Comp
-L Analog_ADC:ADS1115IDGS U4
+L Analog_ADC:ADS1115IDGS U7
 U 1 1 5E458702
 P 5550 3700
-AR Path="/5E1F6B8F/5E458702" Ref="U4"  Part="1"
+AR Path="/5E1F6B8F/5E458702" Ref="U7"  Part="1"
 AR Path="/5E339291/5E458702" Ref="U?"  Part="1"
-F 0 "U4" H 5550 4381 50  0000 C CNN
+F 0 "U7" H 5550 4381 50  0000 C CNN
 F 1 "ADS1115IDGS" H 5550 4290 50  0000 C CNN
 F 2 "Package_SO:TSSOP-10_3x3mm_P0.5mm" H 5550 3200 50  0001 C CNN
